File: fan.kicad_sch (KiCad schematic)
At the start: 15 parts, among them J6 Conn_01x04, U10 EMC2101

Commit message: Powermining upgrades
Parts:
- added J2: Conn_01x04, bitaxe:470531000, symbol Connector_Generic:Conn_01x04
- renumbered R51 to R24
Connections:
- net FAN_PWM: now also J2.4 (Pin_4)
- net FAN_TACH: now also J2.3 (Pin_3)
- net GND: now also J2.1 (Pin_1)
- net at C51.1, C52.1, FB6.2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: now also J2.2 (Pin_2)
Changed lines of the file:
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@@
 (kicad_sch
-	(version 20231120)
+	(version 20250114)
 	(generator "eeschema")
-	(generator_version "8.0")
+	(generator_version "9.0")
 	(paper "A")
 	(title_block
@@
 		(rev "600")
 	)
+	(text "Nerdaxe gamma rev 2.3"
+		(exclude_from_sim no)
+		(at 198.882 178.816 0)
+		(effects
+			(font
+				(size 4 4)
+				(thickness 0.8)
+				(bold yes)
+				(italic yes)
+			)
+		)
+	)
+	(text "EMC2101 Controls the fan, and reads the ASIC chip temperature"
+		(exclude_from_sim no)
+		(at 114.554 53.086 0)
+		(effects
+			(font
+				(size 1.27 1.27)
+			)
+			(justify left bottom)
+		)
+	)
+	(text "This sets default fan speed to 100% ->"
+		(exclude_from_sim no)
+		(at 105.41 106.68 0)
+		(effects
+			(font
+				(size 1.27 1.27)
+			)
+			(justify left bottom)
+		)
+	)
+	(text "I2C Address: 0x4C"
+		(exclude_from_sim no)
+		(at 137.16 90.17 0)
+		(effects
+			(font
+				(size 1.27 1.27)
+			)
+			(justify left bottom)
+		)
+	)
 	(junction
 		(at 82.55 73.66)
@@
 	)
 	(junction
+		(at 165.1 114.3)
+		(diameter 0)
+		(color 0 0 0 0)
+	)
+	(junction
 		(at 82.55 76.2)
 		(diameter 0)
@@
 	)
 	(junction
+		(at 167.64 127)
+		(diameter 0)
+		(color 0 0 0 0)
+	)
+	(junction
 		(at 144.78 127)
 		(diameter 0)
@@
 	(wire
 		(pts
+			(xy 177.8 124.46) (xy 186.69 124.46)
+		)
+		(stroke
+			(width 0)
+			(type default)
+		)
+	)
+	(wire
+		(pts
 			(xy 130.81 66.04) (xy 124.46 66.04)
 		)
@@
 	(wire
 		(pts
+			(xy 165.1 114.3) (xy 165.1 129.54)
+		)
+		(stroke
+			(width 0)
+			(type default)
+		)
+	)
+	(wire
+		(pts
+			(xy 167.64 127) (xy 167.64 132.08)
+		)
+		(stroke
+			(width 0)
+			(type default)
+		)
+	)
+	(wire
+		(pts
 			(xy 144.78 127) (xy 151.13 127)
 		)
@@
 	(wire
 		(pts
+			(xy 177.8 127) (xy 186.69 127)
+		)
+		(stroke
+			(width 0)
+			(type default)
+		)
+	)
+	(wire
+		(pts
 			(xy 179.07 66.04) (xy 191.77 66.04)
 		)
@@
 	(wire
 		(pts
+			(xy 165.1 129.54) (xy 186.69 129.54)
+		)
+		(stroke
+			(width 0)
+			(type default)
+		)
+	)
+	(wire
+		(pts
 			(xy 114.3 81.28) (xy 114.3 86.36)
 		)
@@
 	(wire
 		(pts
-			(xy 151.13 114.3) (xy 179.07 114.3)
+			(xy 151.13 114.3) (xy 165.1 114.3)
 		)
 		(stroke
@@
 	(wire
 		(pts
+			(xy 167.64 132.08) (xy 186.69 132.08)
+		)
+		(stroke
+			(width 0)
+			(type default)
+		)
+	)
+	(wire
+		(pts
 			(xy 134.62 127) (xy 144.78 127)
 		)
@@
 	(wire
 		(pts
+			(xy 165.1 114.3) (xy 179.07 114.3)
+		)
+		(stroke
+			(width 0)
+			(type default)
+		)
+	)
+	(wire
+		(pts
 			(xy 73.66 76.2) (xy 82.55 76.2)
 		)
@@
 			(width 0)
 			(type default)
-		)
-	)
-	(text "Nerdaxe gamma rev 2.3"
-		(exclude_from_sim no)
-		(at 198.882 178.816 0)
-		(effects
-			(font
-				(size 4 4)
-				(thickness 0.8)
-				(bold yes)
-				(italic yes)
-			)
-		)
-	)
-	(text "EMC2101 Controls the fan, and reads the ASIC chip temperature"
-		(exclude_from_sim no)
-		(at 114.554 53.086 0)
-		(effects
-			(font
-				(size 1.27 1.27)
-			)
-			(justify left bottom)
-		)
-	)
-	(text "This sets default fan speed to 100% ->"
-		(exclude_from_sim no)
-		(at 105.41 106.68 0)
-		(effects
-			(font
-				(size 1.27 1.27)
-			)
-			(justify left bottom)
-		)
-	)
-	(text "I2C Address: 0x4C"
-		(exclude_from_sim no)
-		(at 137.16 90.17 0)
-		(effects
-			(font
-				(size 1.27 1.27)
-			)
-			(justify left bottom)
 		)
 	)
 	(label "5V"
 		(at 184.15 66.04 0)
-		(fields_autoplaced yes)
 		(effects
 			(font
@@
 	(label "FAN_PWM"
 		(at 160.02 78.74 0)
-		(fields_autoplaced yes)
 		(effects
 			(font
@@
 	(label "TEMP_DN"
 		(at 120.65 81.28 0)
-		(fields_autoplaced yes)
 		(effects
 			(font
@@
 	(label "GND"
 		(at 160.02 83.82 0)
-		(fields_autoplaced yes)
 		(effects
 			(font
@@
 	(label "TEMP_P"
 		(at 73.66 73.66 0)
-		(fields_autoplaced yes)
 		(effects
 			(font
@@
 	(label "SCL"
 		(at 165.1 73.66 0)
-		(fields_autoplaced yes)
 		(effects
 			(font
@@
 	(label "3V3"
 		(at 147.32 101.6 0)
-		(fields_autoplaced yes)
 		(effects
 			(font
@@
 	(label "FAN_TACH"
 		(at 120.65 83.82 0)
-		(fields_autoplaced yes)
 		(effects
 			(font
@@
 	(label "GND"
 		(at 157.48 127 0)
-		(fields_autoplaced yes)
 		(effects
 			(font
@@
 	(label "FAN_PWM"
 		(at 168.91 109.22 0)
-		(fields_autoplaced yes)
 		(effects
 			(font
@@
 	(label "3V3"
 		(at 110.49 66.04 0)
-		(fields_autoplaced yes)
 		(effects
 			(font
@@
 	(label "5V"
 		(at 132.08 114.3 0)
-		(fields_autoplaced yes)
 		(effects
 			(font
@@
 	(label "GND"
 		(at 119.38 73.66 0)
-		(fields_autoplaced yes)
 		(effects
 			(font
@@
 	(label "SDA"
 		(at 165.1 76.2 0)
-		(fields_autoplaced yes)
 		(effects
 			(font
@@
 	(label "TEMP_DP"
 		(at 120.65 78.74 0)
-		(fields_autoplaced yes)
+		(effects
+			(font
+				(size 1.27 1.27)
+			)
+			(justify left bottom)
+		)
+	)
+	(label "FAN_PWM"
+		(at 177.8 124.46 0)
+		(effects
+			(font
+				(size 1.27 1.27)
+			)
+			(justify left bottom)
+		)
+	)
+	(label "FAN_TACH"
+		(at 177.8 127 0)
 		(effects
 			(font
@@
 	(label "TEMP_N"
 		(at 73.66 76.2 0)
-		(fields_autoplaced yes)
 		(effects
 			(font
@@
 	(label "FAN_TACH"
 		(at 168.91 111.76 0)
-		(fields_autoplaced yes)
 		(effects
 			(font
@@
 		(shape input)
 		(at 129.54 114.3 180)
-		(fields_autoplaced yes)
 		(effects
 			(font
@@
 		(shape input)
 		(at 73.66 73.66 180)
-		(fields_autoplaced yes)
 		(effects
 			(font
@@
 		(shape input)
 		(at 73.66 76.2 180)
-		(fields_autoplaced yes)
 		(effects
 			(font
@@
 		(shape input)
 		(at 171.45 73.66 0)
-		(fields_autoplaced yes)
 		(effects
 			(font
@@
 		(shape input)
 		(at 109.22 66.04 180)
-		(fields_autoplaced yes)
 		(effects
 			(font
@@
 		(shape input)
 		(at 171.45 76.2 0)
-		(fields_autoplaced yes)
 		(effects
 			(font
@@
 		(on_board yes)
 		(dnp no)
-		(property "Reference" "R51"
+		(property "Reference" "R24"
 			(at 151.13 105.41 0)
 			(effects
@@
 					(unit 1)
 				)
+			)
+		)
+	)
+	(symbol
+		(lib_id "Connector_Generic:Conn_01x04")
+		(at 191.77 129.54 0)
+		(mirror x)
+		(unit 1)
+		(exclude_from_sim no)
+		(in_bom yes)
+		(on_board yes)
+		(dnp no)
+		(fields_autoplaced yes)
+		(property "Reference" "J2"
+			(at 191.77 120.015 0)
+			(effects
+				(font
+					(size 1.27 1.27)
+				)
+			)
+		)
+		(property "Value" "Conn_01x04"
+			(at 191.77 120.015 0)
+			(effects
+				(font
+					(size 1.27 1.27)
+				)
+				(hide yes)
+			)
+		)
+		(property "Footprint" "bitaxe:470531000"
+			(at 191.77 129.54 0)
+			(effects
+				(font
+					(size 1.27 1.27)
+				)
+				(hide yes)
+			)
+		)
+		(property "Datasheet" "~"
+			(at 191.77 129.54 0)
+			(effects
+				(font
+					(size 1.27 1.27)
+				)
+				(hide yes)
+			)
+		)
+		(property "Description" ""
+			(at 191.77 129.54 0)
+			(effects
+				(font
+					(size 1.27 1.27)
+				)
+				(hide yes)
+			)
+		)
+		(property "PARTNO" "0470531000"
+			(at 191.77 129.54 0)
+			(effects
+				(font
+					(size 1.27 1.27)
+				)
+				(hide yes)
+			)
+		)
+		(property "DK" "WM4330-ND"
+			(at 191.77 129.54 0)
+			(effects
+				(font
+					(size 1.27 1.27)
+				)
+				(hide yes)
+			)
+		)
+		(pin "1"
+		)
+		(pin "2"
+		)
+		(pin "3"
+		)
+		(pin "4"
+		)
+		(instances
+			(project "nerdaxe-gamma_v2.3"
+				(path "/e63e39d7-6ac0-4ffd-8aa3-1841a4541b55/8e8832ea-6bf1-49d2-b3a5-32a207f555d2"
+					(reference "J2")
+					(unit 1)
+				)
