File: nerdaxe-gamma_v2.3.kicad_pcb (KiCad board)
At the start: 4 copper layers, 60.8 x 99.8 mm, 132 parts, among them J1 54-00164, J6 Conn_01x04, T1 net-tie, U10 EMC2101, U11 T-Display-S3, U2 TPS546D24ARVFR, U5 MCP1824T-1202E/OT, U6 MCP1824T-0802E, U7 25MHz, U8 BM1370_mode1, U9 SN74AVC4T774

Commit message: Powermining upgrades
Parts:
- removed H5, H6, H7, H8: MountingHole, MountingHole:MountingHole_3.5mm
- added ?: LOGO, LOGO, B.Cu at (78.6, 115.8)
- added J2: Conn_01x04, bitaxe:470531000, B.Cu at (109.0, 143.2)
- added MNT1: Mounting_Wuerth_WA-SMSI-M3_H0.5mm_9774005360, Mounting_Wuerth:Mounting_Wuerth_WA-SMSI-M3_H0.5mm_9774005360, B.Cu at (85.1, 96.0)
- added MNT2: Mounting_Wuerth_WA-SMSI-M3_H0.5mm_9774005360, Mounting_Wuerth:Mounting_Wuerth_WA-SMSI-M3_H0.5mm_9774005360, B.Cu at (126.1, 96.0)
- added MNT3: Mounting_Wuerth_WA-SMSI-M3_H0.5mm_9774005360, Mounting_Wuerth:Mounting_Wuerth_WA-SMSI-M3_H0.5mm_9774005360, B.Cu at (85.1, 137.0)
- added MNT4: Mounting_Wuerth_WA-SMSI-M3_H0.5mm_9774005360, Mounting_Wuerth:Mounting_Wuerth_WA-SMSI-M3_H0.5mm_9774005360, B.Cu at (126.1, 137.0)
- moved G*** 30.4 mm to (131.1, 114.3), turned to -90 degrees
- moved U1 6.45 mm to (134.1, 96.6), turned to -90 degrees
- moved C47 0.54 mm to (123.8, 103.6)
- moved C49 0.48 mm to (122.8, 99.7)
- moved FB5 0.38 mm to (124.5, 101.3)
Routing:
- net Net-(J2-Pin_2): track 7.48 -> 23.3 mm
- net /Fan/FAN_PWM: track 32.4 -> 47.4 mm
- net /Fan/FAN_TACH: track 19.9 -> 34.6 mm
- net /3V3: track 161.8 -> 158.0 mm
- net /5V: track 111.7 -> 114.8 mm
- net /BM1370/1V2fb: track 50.3 -> 49.4 mm
- net /SDA: track 154.8 -> 155.8 mm
Other:
- board text added: "rev.2.3PM"
- board text removed: "rev.2.3"
