File: nerdaxe-gamma_v2.3.kicad_sch (KiCad schematic)
At the start: 18 parts, among them J1 54-00164

Commit message: Powermining upgrades
Parts:
- removed H5, H6, H7, H8: MountingHole, MountingHole:MountingHole_3.5mm, symbol Mechanical:MountingHole
