File: power.kicad_sch (KiCad schematic)
At the start: 44 parts, among them T1 net-tie, U2 TPS546D24ARVFR

Commit message: Powermining upgrades
Changed lines of the file:
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@@
 (kicad_sch
-	(version 20231120)
+	(version 20250114)
 	(generator "eeschema")
-	(generator_version "8.0")
+	(generator_version "9.0")
 	(paper "A")
 	(title_block
@@
 		(rev "600")
 	)
+	(text "TPS546D24A is a Buck regulator that steps 4.5-5.5V down to 1.2V @ 20A for the BM1368"
+		(exclude_from_sim no)
+		(at 111.76 17.78 0)
+		(effects
+			(font
+				(size 1.27 1.27)
+			)
+			(justify left bottom)
+		)
+	)
+	(text "https://webench.ti.com/appinfo/webench/scripts/SDP.cgi?ID=3808DBEB40D18F5D"
+		(exclude_from_sim no)
+		(at 152.908 19.304 0)
+		(effects
+			(font
+				(size 1.27 1.27)
+			)
+		)
+	)
+	(text "Input \n4.5-5.5V"
+		(exclude_from_sim no)
+		(at 20.066 48.514 0)
+		(effects
+			(font
+				(size 1.27 1.27)
+			)
+			(justify left bottom)
+		)
+	)
+	(text "Nerdaxe gamma rev 2.3"
+		(exclude_from_sim no)
+		(at 200.66 179.832 0)
+		(effects
+			(font
+				(size 4 4)
+				(thickness 0.8)
+				(bold yes)
+				(italic yes)
+			)
+		)
+	)
+	(text "PGD is an open drain output\nfrom the TPS546D24. Pull up to 3.3V"
+		(exclude_from_sim no)
+		(at 151.13 120.65 0)
+		(effects
+			(font
+				(size 1.27 1.27)
+			)
+			(justify left bottom)
+		)
+	)
+	(text "I2C ADDR = 0x24"
+		(exclude_from_sim no)
+		(at 85.344 91.186 0)
+		(effects
+			(font
+				(size 1.27 1.27)
+			)
+			(justify left bottom)
+		)
+	)
+	(text "Output \n1.2V nominal\n20A max"
+		(exclude_from_sim no)
+		(at 239.522 56.388 0)
+		(effects
+			(font
+				(size 1.27 1.27)
+			)
+			(justify left bottom)
+		)
+	)
+	(text "Connect at\nU3 Pin 37"
+		(exclude_from_sim no)
+		(at 115.57 148.59 0)
+		(effects
+			(font
+				(size 1.27 1.27)
+			)
+			(justify left bottom)
+		)
+	)
 	(junction
 		(at 66.04 90.17)
@@
 		)
 	)
-	(text "TPS546D24A is a Buck regulator that steps 4.5-5.5V down to 1.2V @ 20A for the BM1368"
-		(exclude_from_sim no)
-		(at 111.76 17.78 0)
-		(effects
-			(font
-				(size 1.27 1.27)
-			)
-			(justify left bottom)
-		)
-	)
-	(text "https://webench.ti.com/appinfo/webench/scripts/SDP.cgi?ID=3808DBEB40D18F5D"
-		(exclude_from_sim no)
-		(at 152.908 19.304 0)
-		(effects
-			(font
-				(size 1.27 1.27)
-			)
-		)
-	)
-	(text "Input \n4.5-5.5V"
-		(exclude_from_sim no)
-		(at 20.066 48.514 0)
-		(effects
-			(font
-				(size 1.27 1.27)
-			)
-			(justify left bottom)
-		)
-	)
-	(text "Nerdaxe gamma rev 2.3"
-		(exclude_from_sim no)
-		(at 200.66 179.832 0)
-		(effects
-			(font
-				(size 4 4)
-				(thickness 0.8)
-				(bold yes)
-				(italic yes)
-			)
-		)
-	)
-	(text "PGD is an open drain output\nfrom the TPS546D24. Pull up to 3.3V"
-		(exclude_from_sim no)
-		(at 151.13 120.65 0)
-		(effects
-			(font
-				(size 1.27 1.27)
-			)
-			(justify left bottom)
-		)
-	)
-	(text "I2C ADDR = 0x24"
-		(exclude_from_sim no)
-		(at 85.344 91.186 0)
-		(effects
-			(font
-				(size 1.27 1.27)
-			)
-			(justify left bottom)
-		)
-	)
-	(text "Output \n1.2V nominal\n20A max"
-		(exclude_from_sim no)
-		(at 239.522 56.388 0)
-		(effects
-			(font
-				(size 1.27 1.27)
-			)
-			(justify left bottom)
-		)
-	)
-	(text "Connect at\nU3 Pin 37"
-		(exclude_from_sim no)
-		(at 115.57 148.59 0)
-		(effects
-			(font
-				(size 1.27 1.27)
-			)
-			(justify left bottom)
-		)
-	)
 	(label "GND"
 		(at 134.62 140.97 180)
-		(fields_autoplaced yes)
 		(effects
 			(font
@@
 	(label "PMB_SDA"
 		(at 99.06 101.6 0)
-		(fields_autoplaced yes)
 		(effects
 			(font
@@
 	(label "GND"
 		(at 96.52 74.93 0)
-		(fields_autoplaced yes)
 		(effects
 			(font
@@
 	(label "SW"
 		(at 148.59 39.37 0)
-		(fields_autoplaced yes)
 		(effects
 			(font
@@
 	(label "GND"
 		(at 140.97 77.47 0)
-		(fields_autoplaced yes)
 		(effects
 			(font
@@
 	(label "PMB_SCL"
 		(at 99.06 104.14 0)
-		(fields_autoplaced yes)
 		(effects
 			(font
@@
 	(label "AGND"
 		(at 118.11 128.27 180)
-		(fields_autoplaced yes)
 		(effects
 			(font
@@
 	(label "AGND"
 		(at 72.39 72.39 0)
-		(fields_autoplaced yes)
 		(effects
 			(font
@@
 	(label "GND"
 		(at 207.01 91.44 0)
-		(fields_autoplaced yes)
 		(effects
 			(font
@@
 	(label "PMB_ALRT"
 		(at 99.06 106.68 0)
-		(fields_autoplaced yes)
 		(effects
 			(font
@@
 	(label "PGOOD"
 		(at 147.32 114.3 0)
-		(fields_autoplaced yes)
 		(effects
 			(font
@@
 	(label "GND"
 		(at 72.39 34.29 0)
-		(fields_autoplaced yes)
 		(effects
 			(font
@@
 	(label "AGND"
 		(at 109.22 140.97 0)
-		(fields_autoplaced yes)
 		(effects
 			(font
@@
 	(label "VIN"
 		(at 44.45 17.78 0)
-		(fields_autoplaced yes)
 		(effects
 			(font
@@
 	(label "VDD"
 		(at 217.17 39.37 0)
-		(fields_autoplaced yes)
 		(effects
 			(font
@@
 	(label "3V3"
 		(at 154.94 100.33 0)
-		(fields_autoplaced yes)
 		(effects
 			(font
@@
 		(shape input)
 		(at 238.76 39.37 0)
-		(fields_autoplaced yes)
 		(effects
 			(font
@@
 		(shape output)
 		(at 99.06 106.68 180)
-		(fields_autoplaced yes)
 		(effects
 			(font
@@
 		(shape input)
 		(at 154.94 100.33 180)
-		(fields_autoplaced yes)
 		(effects
 			(font
@@
 		(shape input)
 		(at 99.06 104.14 180)
-		(fields_autoplaced yes)
 		(effects
 			(font
@@
 		(shape output)
 		(at 172.72 114.3 0)
-		(fields_autoplaced yes)
 		(effects
 			(font
@@
 		(shape input)
 		(at 99.06 101.6 180)
-		(fields_autoplaced yes)
 		(effects
 			(font
@@
 		(shape output)
 		(at 105.41 17.78 0)
-		(fields_autoplaced yes)
 		(effects
 			(font
@@
 		(shape input)
 		(at 21.59 17.78 180)
-		(fields_autoplaced yes)
 		(effects
 			(font
@@
 		)
 	)
+	(embedded_fonts no)
 )
